Commit message: End of Assignment 5

File: body.urdf (robot description, URDF)
Before this commit: robot robot, 3 links, 2 joints
Links:
- removed link Left_Leg
- removed link Right_Leg
- added link Back_Leg, mass 1; collision box size=1 1 1; visual box size=1 1 1
- added link Front_Leg, mass 1; collision box size=1 1 1; visual box size=1 1 1
Joints:
- removed joint Torso_Left_Leg
- removed joint Torso_Right_Leg
- added joint Torso_Back_Leg: type revolute, parent Torso, child Back_Leg, origin xyz=-.5 0 1 rpy=0 0 0, axis 0 1 0, limit lower=-3.14159 upper=3.14159 effort=0.0 velocity=0.0
- added joint Torso_Front_Leg: type revolute, parent Torso, child Front_Leg, origin xyz=.5 0 1 rpy=0 0 0, axis 0 1 0, limit lower=-3.14159 upper=3.14159 effort=0.0 velocity=0.0

Commit message: Done with quadruped

File: body.urdf (robot description, URDF)
Before this commit: robot robot, 3 links, 2 joints
Links:
- added link Left_Leg, mass 1; collision box size=1 0.2 0.2; visual box size=1 0.2 0.2
- added link Lower_Back_Leg, mass 1; collision box size=0.2 0.2 1; visual box size=0.2 0.2 1
- added link Lower_Front_Leg, mass 1; collision box size=0.2 0.2 1; visual box size=0.2 0.2 1
- added link Lower_Left_Leg, mass 1; collision box size=0.2 0.2 1; visual box size=0.2 0.2 1
- added link Lower_Right_Leg, mass 1; collision box size=0.2 0.2 1; visual box size=0.2 0.2 1
- added link Right_Leg, mass 1; collision box size=1 0.2 0.2; visual box size=1 0.2 0.2
- link Back_Leg: geometry collision box size=0.2 1 0.2; visual box size=0.2 1 0.2
- link Front_Leg: geometry collision box size=0.2 1 0.2; visual box size=0.2 1 0.2
Joints:
- added joint Back_Leg_Lower_Back_Leg: type revolute, parent Back_Leg, child Lower_Back_Leg, origin xyz=0 -1 0 rpy=0 0 0, axis 0 0 1, limit lower=-3.14159 upper=3.14159 effort=0.0 velocity=0.0
- added joint Front_Leg_Lower_Front_Leg: type revolute, parent Front_Leg, child Lower_Front_Leg, origin xyz=0 1 0 rpy=0 0 0, axis 0 0 1, limit lower=-3.14159 upper=3.14159 effort=0.0 velocity=0.0
- added joint Left_Leg_Lower_Left_Leg: type revolute, parent Left_Leg, child Lower_Left_Leg, origin xyz=-1 -.5 -.5 rpy=0 0 0, axis 0 0 1, limit lower=-3.14159 upper=3.14159 effort=0.0 velocity=0.0
- added joint Right_Leg_Lower_Right_Leg: type revolute, parent Right_Leg, child Lower_Right_Leg, origin xyz=1 0 -.5 rpy=0 0 0, axis 0 0 1, limit lower=-3.14159 upper=3.14159 effort=0.0 velocity=0.0
- added joint Torso_Left_Leg: type revolute, parent Torso, child Left_Leg, origin xyz=-.5 0 1 rpy=0 0 0, axis 0 1 0, limit lower=-3.14159 upper=3.14159 effort=0.0 velocity=0.0
- added joint Torso_Right_Leg: type revolute, parent Torso, child Right_Leg, origin xyz=.5 0 1 rpy=0 0 0, axis 0 1 0, limit lower=-3.14159 upper=3.14159 effort=0.0 velocity=0.0
- joint Torso_Back_Leg: axis 0 1 0 -> 1 0 0; origin xyz=-.5 0 1 rpy=0 0 0 -> xyz=0 -.5 1 rpy=0 0 0
- joint Torso_Front_Leg: axis 0 1 0 -> 1 0 0; origin xyz=.5 0 1 rpy=0 0 0 -> xyz=0 .5 1 rpy=0 0 0
